File: TKKB.kicad_pcb (KiCad board)
At the start: 2 copper layers, 65 parts, among them J1 UP, J2 DOWN, J3 Power Connector, SW1 RESET, SW10 6, SW11 7, SW12 8, SW13 9, SW14 0, SW15 1, SW16 Q, SW17 W, SW18 E, SW19 R, SW2 REPEAT, SW20 T, SW21 Y, SW22 U, SW23 I, SW24 O, SW25 P, SW26 FIRE, SW27 FIRE, SW28 UP, SW29 DOWN, SW3 SPACE, SW30 RETURN, SW31 CTRL, SW32 A, SW33 S, SW34 D, SW35 F, SW36 G, SW37 H, SW38 J, SW39 K, SW4 SPACE, SW40 L, SW41 :, SW42 LEFT, SW43 RIGHT, SW44 SHIFT, SW45 SHIFT, SW46 Z, SW47 X, SW48 C, SW49 V, SW5 SPACE, SW50 B, SW51 N, SW52 M, SW53 ,, SW54 ., SW55 ?, SW6 2, SW7 3, SW8 4, SW9 5

Commit message: Created the base keyboard
Parts:
- added SW56: RETURN, buttons:SW_Push_SMD_Large, F.Cu at (208.3, 81.3)
- added SW57: CTRL, buttons:SW_Push_SMD_Large, F.Cu at (210.8, 111.8)
- H1, H2, H3, H4, H5, H6: footprint MountingHole:MountingHole_3.2mm_M3_Pad -> MountingHole:MountingHole_3.2mm_M3_ISO7380
- J1: footprint Connector_PinHeader_2.54mm:PinHeader_1x08_P2.54mm_Horizontal -> Connector_PinHeader_2.54mm:PinHeader_1x08_P2.54mm_Vertical
- J2: footprint Connector_PinHeader_2.54mm:PinHeader_1x13_P2.54mm_Horizontal -> Connector_PinHeader_2.54mm:PinHeader_1x13_P2.54mm_Vertical
- J3: footprint Connector_PinHeader_2.54mm:PinHeader_1x02_P2.54mm_Horizontal -> Connector_PinHeader_2.54mm:PinHeader_1x02_P2.54mm_Vertical
- moved SW1 154.2 mm to (259.1, 81.3)
- moved H2 141.3 mm to (35.6, 129.5)
- moved H1 137.2 mm to (35.6, 68.6)
- moved SW2 122.8 mm to (228.6, 81.3)
- moved SW46 116.6 mm to (58.4, 111.8), turned to 180 degrees
- moved SW29 112.2 mm to (243.8, 121.9), turned to 180 degrees
- moved SW28 111.7 mm to (243.8, 111.8), turned to 180 degrees
- moved SW43 111.1 mm to (259.1, 121.9), turned to 180 degrees
- moved SW44 110.2 mm to (40.6, 101.6), turned to 180 degrees
- moved SW47 99.5 mm to (73.7, 111.8), turned to 180 degrees
- moved J3 99.3 mm to (241.1, 67.9), turned to 90 degrees
- moved D1 98.7 mm to (242.4, 71.1), turned to 180 degrees
- moved SW27 97.3 mm to (38.1, 91.4), turned to 180 degrees
- moved SW31 91.6 mm to (43.2, 111.8), turned to 180 degrees
- moved H6 85.1 mm to (264.2, 129.5)
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Connections:
- SW3 pad 1: /O1 -> /O3
- SW4 pad 1: /O1 -> /O3
- SW5 pad 1: unconnected-(SW5-Pad1) -> /O3
Routing:
- net /I0: track 0.00 -> 372.9 mm, vias 0 -> 12
- net /O7: track 0.00 -> 324.6 mm, vias 0 -> 8
- net /I4: track 0.00 -> 312.8 mm, vias 0 -> 9
- net /I1: track 0.00 -> 284.2 mm, vias 0 -> 6
- net /I5: track 0.00 -> 281.7 mm, vias 0 -> 11
- net /O8: track 0.00 -> 255.0 mm, vias 0 -> 5
- net /O1: track 0.00 -> 240.9 mm, vias 0 -> 3
- net /I3: track 0.00 -> 223.7 mm, vias 0 -> 9
- net /O6: track 0.00 -> 220.4 mm, vias 0 -> 1
- net /O0: track 0.00 -> 213.2 mm, vias 0 -> 4
- net /I2: track 0.00 -> 206.9 mm, vias 0 -> 10
- net /O3: track 0.00 -> 206.8 mm, vias 0 -> 5
- net /O2: track 0.00 -> 204.4 mm, vias 0 -> 3
- net /O4: track 0.00 -> 194.4 mm, vias 0 -> 3
- net /~{RESET}: track 0.00 -> 164.8 mm, vias 0 -> 3
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Other:
- board outline added: 238.8 x 71.1 mm
