File: TKKB.kicad_pcb (KiCad board)
At the start: 2 copper layers, 238.8 x 71.1 mm, 67 parts, among them J1 UP, J2 DOWN, J3 Power Connector, SW1 RESET, SW10 6, SW11 7, SW12 8, SW13 9, SW14 0, SW15 1, SW16 Q, SW17 W, SW18 E, SW19 R, SW2 REPEAT, SW20 T, SW21 Y, SW22 U, SW23 I, SW24 O, SW25 P, SW26 FIRE, SW27 FIRE, SW28 UP, SW29 DOWN, SW3 SPACE, SW30 RETURN, SW31 CTRL, SW32 A, SW33 S, SW34 D, SW35 F, SW36 G, SW37 H, SW38 J, SW39 K, SW4 SPACE, SW40 L, SW41 :, SW42 LEFT, SW43 RIGHT, SW44 SHIFT, SW45 SHIFT, SW46 Z, SW47 X, SW48 C, SW49 V, SW5 SPACE, SW50 B, SW51 N, SW52 M, SW53 ,, SW54 ., SW55 ?, SW56 RETURN, SW57 CTRL, SW6 2, SW7 3, SW8 4, SW9 5

Commit message: Add silkscreen for every key
Parts:
- D1: footprint LED_SMD:LED_1206_3216Metric_Pad1.42x1.75mm_HandSolder -> LED_THT:LED_D3.0mm
- SW41: value : -> : ;
- SW53: value , -> , <
- SW54: value . -> . >
- SW55: value ? -> ? /
- moved D1 1.63 mm to (243.6, 72.1)
Routing:
- net Net-(D1-K): track 3.34 -> 4.58 mm
- net Net-(D1-A): track 3.34 -> 4.27 mm
Other:
- board text added: "↩️"
- board text added: "➡️"
- board text added: "⬅️"
- board text added: "⬆️"
- board text added: "⬇️"

Commit message: Add rev.0 gerbers
Other:
- board text added: "Rev. 0"
- board text added: "TK2KB"
Changed lines of the file:
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@@
 			(outputformat 1)
 			(mirror no)
-			(drillshape 1)
+			(drillshape 0)
 			(scaleselection 1)
-			(outputdirectory "")
+			(outputdirectory "gerbers/")
 		)
 	)
@@
 		(layer "Edge.Cuts")
 	)
+	(gr_text "TK2KB"
+		(at 39.878 129.54 0)
+		(layer "F.Cu")
+		(effects
+			(font
+				(size 4 4)
+				(thickness 0.8)
+				(bold yes)
+			)
+			(justify left)
+		)
+	)
+	(gr_text "Rev. 0"
+		(at 59.69 130.81 0)
+		(layer "F.Cu")
+		(effects
+			(font
+				(size 1.5 1.5)
+				(thickness 0.3)
+				(bold yes)
+			)
+			(justify left)
+		)
+	)
+	(gr_text "Rev. 0"
+		(at 59.69 130.81 0)
+		(layer "F.Mask")
+		(effects
+			(font
+				(size 1.5 1.5)
+				(thickness 0.3)
+				(bold yes)
+			)
+			(justify left)
+		)
+	)
+	(gr_text "TK2KB"
+		(at 39.878 129.54 0)
+		(layer "F.Mask")
+		(effects
+			(font
+				(size 4 4)
+				(thickness 0.8)
+				(bold yes)
+			)
+			(justify left)
+		)
+	)
 	(gr_text "⬆️"

Commit message: Add more stand holes for the keyboard
Parts:
- added H10: MountingHole_Pad, MountingHole:MountingHole_3.2mm_M3_ISO7380, F.Cu at (231.1, 68.6)
- added H7: MountingHole_Pad, MountingHole:MountingHole_3.2mm_M3_ISO7380, F.Cu at (92.7, 129.5)
- added H8: MountingHole_Pad, MountingHole:MountingHole_3.2mm_M3_ISO7380, F.Cu at (207.0, 129.5)
- added H9: MountingHole_Pad, MountingHole:MountingHole_3.2mm_M3_ISO7380, F.Cu at (68.8, 68.6)
